File: Epic-Laser/Epic-Laser.kicad_sch (KiCad schematic)
At the start: 0 parts

Commit message: Draft-Schematics
Parts:
- added C1, C2, C4: 10u, Capacitor_THT:C_Disc_D5.0mm_W2.5mm_P2.50mm, symbol Device:C_Small
- added C3, C5: 100n, Capacitor_THT:C_Disc_D5.0mm_W2.5mm_P2.50mm, symbol Device:C_Small
- added CR1: LD1117V33, SnapMagic-Footprints:TO-220_STM, symbol 2026-04-24_23-55-40:LD1117V33
- added D1: LED, symbol Device:LED
- added J1: ICSP-Header, Connector_PinSocket_2.54mm:PinSocket_1x07_P2.54mm_Vertical, symbol Connector:Conn_01x06_Socket
- added J2: X-Motor, symbol Connector:Conn_01x05_Socket
- added J3: Y-Motor, symbol Connector:Conn_01x05_Socket
- added J4: Laser_Control, symbol Connector:Screw_Terminal_01x02
- added Q1: 2N7000, Package_TO_SOT_THT:TO-92_Inline, symbol Transistor_FET:2N7000
- added R1: 10k, Resistor_THT:R_Axial_DIN0204_L3.6mm_D1.6mm_P5.08mm_Horizontal, symbol Device:R_Small_US
- added R2: 1k, symbol Device:R_Small_US
- added U1: PIC24FJ64GA002-I_SP, SnapMagic-Footprints:DIP787W46P254L3467H508Q28, symbol PIC24FJ64GA002-I_SP:PIC24FJ64GA002-I_SP
- added X1: USB-B1HSB6, SnapMagic-Footprints:OST_USB-B1HSB6, symbol USB-B1HSB6:USB-B1HSB6
Connections:
- new net: D1.2 (A), R2.1
- new net: C1.1, U1.20 (VCAP/VDDCORE)
- new net: J4.1 (Pin_1), Q1.3 (D)
- new net +3.3V: C2.2, C3.2, C4.2, CR1.2 (VOUT), J1.2 (Pin_2), J2.1 (Pin_1), J3.1 (Pin_1), R1.1, R2.2, U1.13 (VDD), U1.28 (VDD)
- new net +5V: C5.2, CR1.3 (VIN), J4.2 (Pin_2), X1.1 (VCC)
- new net GND: C1.2, C2.1, C3.1, C4.1, C5.1, CR1.1 (ADJ/GND), D1.1 (K), J1.3 (Pin_3), J2.2 (Pin_2), J3.2 (Pin_2), Q1.1 (S), U1.19 (DISVREG), U1.27 (VSS), U1.8 (VSS), X1.4 (GND)
- new net Laser_Drive: Q1.2 (G)
- new net PGC1: J1.5 (Pin_5), U1.5 (PGC1/EMUC1/AN3/C2IN+/RP1/CN5/RB1)
- new net PGD1: J1.4 (Pin_4), U1.4 (PGD1/EMUD1/AN2/C2IN-/RP0/CN4/RB0)
- new net X_DIR: J2.4 (Pin_4), U1.17 (TCK/RP8/SCL1/CN22/PMD4/RB8)
- new net X_EN: J2.5 (Pin_5), J3.5 (Pin_5), U1.21 (PGD2/EMUD2/TDI/RP10/CN16/PMD2/RB10)
- new net X_STEP: J2.3 (Pin_3), U1.15 (PGC3/EMUC3/RP6/ASCL1/CN24/PMD6/RB6)
- new net Y_DIR: J3.4 (Pin_4), U1.18 (TDO/RP9/SDA1/CN21/PMD3/RB9)
- new net Y_STEP: J3.3 (Pin_3), U1.16 (RP7/INT0/CN23/PMD5/RB7)
- new net nMCLR: J1.1 (Pin_1), R1.2, U1.1 (~{MCLR})
- no-connect marks 0 -> 17
Other:
- company: (none) -> Epic Laser Corp
- title: (none) -> Vector-Display-Controller
